Commit message: Imported upstream version '0.3.1' of 'upstream'

File: hector_sensors_description/urdf/hokuyo_utm30lx.urdf.xacro (robot description, xacro)
@@ -2,5 +2,5 @@
 <robot xmlns:xacro="http://ros.org/wiki/xacro">
     <xacro:property name="M_PI" value="3.1415926535897931" />
-    <xacro:macro name="hokuyo_utm30lx" params="name parent *origin ros_topic update_rate ray_count min_angle max_angle">
+    <xacro:macro name="hokuyo_utm30lx_model" params="name parent *origin">
       <joint name="${name}_joint" type="fixed">
         <xacro:insert_block name="origin" />
@@ -28,4 +28,9 @@
         </collision>
       </link>
+    </xacro:macro>
+    <xacro:macro name="hokuyo_utm30lx" params="name parent *origin ros_topic update_rate ray_count min_angle max_angle">
+      <xacro:hokuyo_utm30lx_model name="${name}" parent="${parent}">
+        <xacro:insert_block name="origin" />
+      </xacro:hokuyo_utm30lx_model>
       <gazebo reference="${name}_frame">
         <sensor type="ray" name="${name}">
@@ -59,3 +64,38 @@
       </gazebo>
     </xacro:macro>
-  </robot>
+    <xacro:macro name="hokuyo_utm30lx_gpu" params="name parent *origin ros_topic update_rate ray_count min_angle max_angle">
+      <xacro:hokuyo_utm30lx_model name="${name}" parent="${parent}">
+        <xacro:insert_block name="origin" />
+      </xacro:hokuyo_utm30lx_model>
+      <gazebo reference="${name}_frame">
+        <sensor type="gpu_ray" name="${name}">
+          <always_on>true</always_on>
+          <update_rate>${update_rate}</update_rate>
+          <pose>0 0 0 0 0 0</pose>
+          <visualize>false</visualize>
+          <ray>
+            <scan>
+              <horizontal>
+                <samples>${ray_count}</samples>
+                <resolution>1</resolution>
+                <min_angle>${min_angle * M_PI/180}</min_angle>
+                <max_angle>${max_angle * M_PI/180}</max_angle>
+              </horizontal>
+            </scan>
+            <range>
+              <min>0.08</min>
+              <max>30.0</max>
+              <resolution>0.01</resolution>
+            </range>
+          </ray>
+          <plugin name="gazebo_ros_${name}_controller" filename="libgazebo_ros_gpu_laser.so">
+            <gaussianNoise>0.005</gaussianNoise>
+            <alwaysOn>true</alwaysOn>
+            <updateRate>${update_rate}</updateRate>
+            <topicName>${ros_topic}</topicName>
+            <frameName>${name}_frame</frameName>
+          </plugin>
+        </sensor>
+      </gazebo>
+    </xacro:macro>
+</robot>
