Commit message: Imported upstream version '0.5.0' of 'upstream'

File: hector_sensors_description/urdf/flir_a35_camera.urdf.xacro (robot description, xacro)
@@ -1,4 +1,4 @@
 <?xml version="1.0"?>
-<robot xmlns:xacro="http://www.ros.org/wiki/xacro">
+<robot xmlns:xacro="http://ros.org/wiki/xacro">
   <xacro:include filename="$(find hector_xacro_tools)/urdf/sensor_macros.urdf.xacro" />
   <xacro:macro name="flir_a35_camera_model" params="name parent *origin">
@@ -55,6 +55,7 @@
           <alwaysOn>true</alwaysOn>
           <updateRate>10</updateRate>
-          <imageTopicName>/${name}/image</imageTopicName>
-          <cameraInfoTopicName>/${name}/camera_info</cameraInfoTopicName>
+          <cameraName>${name}</cameraName>
+          <imageTopicName>image_raw</imageTopicName>
+          <cameraInfoTopicName>camera_info</cameraInfoTopicName>
           <frameName>${name}_optical_frame</frameName>
         </plugin>

File: hector_sensors_description/urdf/generic_thermal_camera.urdf.xacro (robot description, xacro)
@@ -1,4 +1,4 @@
 <?xml version="1.0"?>
-<robot xmlns:xacro="http://www.ros.org/wiki/xacro">
+<robot xmlns:xacro="http://ros.org/wiki/xacro">
   <xacro:include filename="$(find hector_xacro_tools)/urdf/sensor_macros.urdf.xacro" />
   <xacro:macro name="generic_thermal_camera" params="name parent *origin">
@@ -31,6 +31,6 @@
           <image>
             <format>R8G8B8</format>
-            <width>160</width>
-            <height>120</height>
+            <width>320</width>
+            <height>256</height>
           </image>
           <clip>
@@ -42,5 +42,5 @@
           <alwaysOn>true</alwaysOn>
           <updateRate>10</updateRate>
-          <imageTopicName>/${name}/image</imageTopicName>
+          <imageTopicName>/${name}/image_raw</imageTopicName>
           <cameraInfoTopicName>/${name}/camera_info</cameraInfoTopicName>
           <frameName>${name}_optical_frame</frameName>

File: hector_sensors_description/urdf/kinect_camera.urdf.xacro (robot description, xacro)
@@ -1,4 +1,5 @@
 <?xml version="1.0"?>
-<robot xmlns:xacro="http://www.ros.org/wiki/xacro">
+<robot xmlns:xacro="http://ros.org/wiki/xacro">
+    <xacro:include filename="$(find hector_xacro_tools)/urdf/inertia_tensors.urdf.xacro"/>
     <xacro:property name="M_PI" value="3.1415926535897931" />
     <xacro:macro name="kinect_camera_model" params="name parent *origin">
@@ -58,5 +59,5 @@
             <horizontal_fov>${60 * M_PI/180.0}</horizontal_fov>
             <image>
-              <format>R8G8B8</format>
+              <format>B8G8R8</format>
               <width>640</width>
               <height>480</height>

File: hector_sensors_description/urdf/realsense_d435_camera.urdf.xacro (robot description, xacro)
@@ -14,5 +14,5 @@
      the openni gazebo plugin. See the 'asus_camera' macro below for that
     -->
-    <xacro:macro name="realsense_camera_model" params="name parent *origin">
+    <xacro:macro name="realsense_d435_camera_model" params="name parent *origin">
       <joint name="${name}_joint" type="fixed">
         <xacro:insert_block name="origin" />
@@ -22,13 +22,13 @@
       <link name="${name}_link">
         <inertial>
-          <mass value="0.200" />
+          <mass value="0.072" />
           <origin xyz="0 0 0" rpy="0 0 0" />
           <inertia ixx="5.8083e-4" ixy="0" ixz="0" iyy="3.0833e-5" iyz="0" izz="5.9083e-4" />
         </inertial>
         <visual>
-          <origin xyz="0 0.051 0" rpy="0 0 0" />
+          <origin xyz="0 0.0115 0" rpy="0 0 0" />
           <geometry>
-            <!--Dimensions taken from https://software.intel.com/en-us/realsense/devkit-->
-            <box size="0.007 0.130 0.02" />
+            <!--Dimensions taken from https://click.intel.com/intelr-realsensetm-depth-camera-d435.html-->
+            <box size="0.025 0.09 0.025" />
           </geometry>
           <material name="DarkGrey">
@@ -37,54 +37,16 @@
         </visual>
         <collision>
-          <origin xyz="0 0.051 0" rpy="0 0 0" />
+          <origin xyz="0 0.0115 0" rpy="0 0 0" />
           <geometry>
-            <!--Dimensions taken from https://software.intel.com/en-us/realsense/devkit-->
-            <box size="0.007 0.130 0.02" />
-          </geometry>
+            <!--Dimensions taken from https://click.intel.com/intelr-realsensetm-depth-camera-d435.html-->
+            <box size="0.025 0.09 0.025" />
+          </geometry>update_rate
         </collision>
       </link>
-      <!--
-      <joint name="${name}_depth_joint" type="fixed">
-        <origin xyz="0 -0.051 0.004" rpy="0 0 0" />
-        <parent link="${name}_link" />
-        <child link="${name}_depth_frame"/>
-      </joint>
-      <link name="${name}_depth_frame"/>
-      <joint name="${name}_depth_optical_joint" type="fixed">
-        <origin xyz="0 0 0" rpy="${-M_PI/2} 0.0 ${-M_PI/2}" />
-        <parent link="${name}_depth_frame" />
-        <child link="${name}_depth_optical_frame"/>
-      </joint>
-      <link name="${name}_depth_optical_frame"/>
-      <joint name="${name}_depth_joint_aux" type="fixed">
-        <origin xyz="0 0.032 0.004" rpy="0 0 0" />
-        <parent link="${name}_link" />
-        <child link="${name}_depth_frame_aux"/>
-      </joint>
-      <link name="${name}_depth_frame_aux"/>
-      <joint name="${name}_depth_optical_joint_aux" type="fixed">
-        <origin xyz="0 0 0" rpy="${-M_PI/2} 0.0 ${-M_PI/2}" />
-        <parent link="${name}_depth_frame_aux" />
-        <child link="${name}_depth_optical_frame_aux"/>
-      </joint>
-      <link name="${name}_depth_optical_frame_aux"/>
-      <joint name="${name}_rgb_joint" type="fixed">
-        <origin xyz="0 -0.045 0.004" rpy="0 0 0" />
-        <parent link="${name}_link" />
-        <child link="${name}_rgb_frame"/>
-      </joint>
-      <link name="${name}_rgbd_cam_link"/>
-      <joint name="${name}_rgb_optical_joint" type="fixed">
-        <origin xyz="0 0 0" rpy="${-M_PI/2} 0.0 ${-M_PI/2}" />
-        <parent link="${name}_rgb_frame" />
-        <child link="${name}_rgb_optical_frame"/>
-      </joint>
-      <link name="${name}_rgb_optical_frame"/>
-      -->
       <gazebo reference="${name}_link">
         <material>Gazebo/Grey</material>
       </gazebo>
     </xacro:macro>
-    <xacro:macro name="realsense_camera_model_no_geom" params="name parent *origin">
+    <xacro:macro name="realsense_d435_camera_model_no_geom" params="name parent *origin">
       <joint name="${name}_joint" type="fixed">
         <xacro:insert_block name="origin" />
@@ -95,13 +57,13 @@
       </link>
     </xacro:macro>
-    <xacro:macro name="realsense_camera_gazebo_plugin_macro" params="name parent image_topic depth_points_topic min_range max_range update_rate">
+    <xacro:macro name="realsense_d435_camera_gazebo_plugin_macro" params="name parent image_topic depth_points_topic min_range max_range update_rate">
       <gazebo reference="${name}_link">
         <sensor type="depth" name="${name}">
           <update_rate>${update_rate}</update_rate>
           <camera>
-            <horizontal_fov>${53.35 * M_PI/180.0}</horizontal_fov>
+            <horizontal_fov>${69.4 * M_PI/180.0}</horizontal_fov>
             <image>
               <format>B8G8R8</format>
-              <width>640</width>
+              <width>848</width>
               <height>480</height>
             </image>
@@ -126,9 +88,9 @@
       Use the macro below for adding the realsense model with link geometry
     -->
-    <xacro:macro name="realsense_camera" params="name parent *origin">
-      <xacro:realsense_camera_model name="${name}" parent="${parent}">
+    <xacro:macro name="realsense_d435_camera" params="name parent *origin">
+      <xacro:realsense_d435_camera_model name="${name}" parent="${parent}">
         <xacro:insert_block name="origin" />
-      </xacro:realsense_camera_model>
-      <xacro:realsense_camera_gazebo_plugin_macro name="${name}" parent="${parent}" image_topic="rgb/image_raw" depth_points_topic="depth/points" min_range="0.3" max_range="9.0" update_rate="20"/>
+      </xacro:realsense_d435_camera_model>
+      <xacro:realsense_d435_camera_gazebo_plugin_macro name="${name}" parent="${parent}" image_topic="rgb/image_raw" depth_points_topic="depth/points" min_range="0.3" max_range="9.0" update_rate="20"/>
     </xacro:macro>
     <!--
@@ -137,20 +99,20 @@
     -->
     <xacro:macro name="realsense_camera_no_geom" params="name parent *origin">
-      <xacro:realsense_camera_model_no_geom name="${name}" parent="${parent}">
+      <xacro:realsense_d435_camera_model_no_geom name="${name}" parent="${parent}">
         <xacro:insert_block name="origin" />
-      </xacro:realsense_camera_model_no_geom>
+      </xacro:realsense_d435_camera_model_no_geom>
       <xacro:realsense_camera_gazebo_plugin_macro name="${name}" parent="${parent}" image_topic="rgb/image_raw" depth_points_topic="depth/points" min_range="0.3" max_range="9.0" update_rate="20"/>
     </xacro:macro>
-    <xacro:macro name="realsense_camera_no_geom_comprehensive_params" params="name parent *origin image_topic depth_points_topic min_range max_range update_rate">
-      <xacro:realsense_camera_model_no_geom name="${name}" parent="${parent}">
+    <xacro:macro name="realsense_d435_camera_no_geom_comprehensive_params" params="name parent *origin image_topic depth_points_topic min_range max_range update_rate">
+      <xacro:realsense_d435_camera_model_no_geom name="${name}" parent="${parent}">
         <xacro:insert_block name="origin" />
-      </xacro:realsense_camera_model_no_geom>
+      </xacro:realsense_d435_camera_model_no_geom>
       <xacro:realsense_camera_gazebo_plugin_macro name="${name}" parent="${parent}" image_topic="${image_topic}" depth_points_topic="${depth_points_topic}" min_range="${min_range}" max_range="${max_range}" update_rate="${update_rate}"/>
     </xacro:macro>
-    <xacro:macro name="realsense_camera_comprehensive_params" params="name parent *origin image_topic depth_points_topic min_range max_range update_rate">
-      <xacro:realsense_camera_model name="${name}" parent="${parent}">
+    <xacro:macro name="realsense_d435_camera_comprehensive_params" params="name parent *origin image_topic depth_points_topic min_range max_range update_rate">
+      <xacro:realsense_d435_camera_model name="${name}" parent="${parent}">
         <xacro:insert_block name="origin" />
-      </xacro:realsense_camera_model>
-      <xacro:realsense_camera_gazebo_plugin_macro name="${name}" parent="${parent}" image_topic="${image_topic}" depth_points_topic="${depth_points_topic}" min_range="${min_range}" max_range="${max_range}" update_rate="${update_rate}"/>
+      </xacro:realsense_d435_camera_model>
+      <xacro:realsense_d435_camera_gazebo_plugin_macro name="${name}" parent="${parent}" image_topic="${image_topic}" depth_points_topic="${depth_points_topic}" min_range="${min_range}" max_range="${max_range}" update_rate="${update_rate}"/>
     </xacro:macro>
   </robot>

File: hector_sensors_description/urdf/vlp16.urdf.xacro (robot description, xacro)
@@ -2,5 +2,5 @@
 <robot xmlns:xacro="http://ros.org/wiki/xacro">
     <xacro:property name="M_PI" value="3.1415926535897931" />
-    <xacro:macro name="hokuyo_utm30lx_model" params="name parent *origin">
+    <xacro:macro name="vlp16_model" params="name parent *origin">
       <joint name="${name}_joint" type="fixed">
         <xacro:insert_block name="origin" />
@@ -9,30 +9,30 @@
       </joint>
       <link name="${name}_frame">
-        <inertial>
-          <mass value="0.270" />
-          <origin xyz="0 0 0" rpy="0 0 0" />
-          <inertia ixx="2.632e-4" ixy="0" ixz="0" iyy="2.632e-4" iyz="0" izz="1.62e-4" />
-        </inertial>
-        <visual>
-          <origin xyz="0 0 0" rpy="0 0 0" />
+        <xacro:inertial_sphere mass="0.8" diameter="0.1033" />
+        <visual>        -->
+          <origin rpy="0 0 0" xyz="0 0 0.0018500"/>
           <geometry>
-          <mesh filename="package://hector_sensors_description/meshes/hokuyo_utm30lx/hokuyo_utm_30lx$(optenv TEST_SELF_FILTER).dae"/>
-        </geometry>
+            <cylinder radius="0.0516" length="0.0717"/>
+          </geometry>
         </visual>
         <collision>
-          <origin xyz="0 0 -0.0115" rpy="0 0 0" />
+          <origin rpy="0 0 0" xyz="0 0 0.0018500"/>
           <geometry>
-          <box size="0.058 0.058 0.087" />
-          <!--<mesh filename="package://hector_sensors_description/meshes/hokuyo_utm30lx/hokuyo_utm_30lx.stl"/>-->
-        </geometry>
+            <cylinder radius="0.0516" length="0.0717"/>
+          </geometry>
         </collision>
       </link>
     </xacro:macro>
-    <xacro:macro name="hokuyo_utm30lx" params="name parent *origin ros_topic update_rate ray_count min_angle max_angle">
-      <xacro:hokuyo_utm30lx_model name="${name}" parent="${parent}">
+    <xacro:macro name="vlp16" params="name parent *origin ros_topic">
+      <xacro:vlp16_advanced_parameters name="${name}" parent="${parent}" ros_topic="${ros_topic}" update_rate="10" horizontal_samples="512" vertical_samples="8" min_range="0.45" max_range="100">
         <xacro:insert_block name="origin" />
-      </xacro:hokuyo_utm30lx_model>
+      </xacro:vlp16_advanced_parameters>
+    </xacro:macro>
+    <xacro:macro name="vlp16_advanced_parameters" params="name parent *origin ros_topic update_rate horizontal_samples vertical_samples min_range max_range">
+      <xacro:vlp16_model name="${name}" parent="${parent}">
+        <xacro:insert_block name="origin" />
+      </xacro:vlp16_model>
       <gazebo reference="${name}_frame">
-        <sensor type="ray" name="${name}">
+<!--        <sensor type="ray" name="${name}">
           <always_on>true</always_on>
           <update_rate>${update_rate}</update_rate>
@@ -63,11 +63,49 @@
             <frameName>${name}_frame</frameName>
           </plugin>
-        </sensor>
+        </sensor>-->
+      <sensor type="ray" name="${name}-VLP16">
+        <pose>0 0 0 0 0 0</pose>
+        <visualize>false</visualize>
+        <update_rate>${update_rate}</update_rate>
+        <ray>
+          <scan>
+            <horizontal>
+              <samples>${horizontal_samples}</samples>
+              <resolution>1</resolution>
+              <min_angle>-${M_PI}</min_angle>
+              <max_angle> ${M_PI}</max_angle>
+            </horizontal>
+            <vertical>
+              <samples>${vertical_samples}</samples>
+              <resolution>1</resolution>
+              <min_angle>-${15.0*M_PI/180.0}</min_angle>
+              <max_angle> ${15.0*M_PI/180.0}</max_angle>
+            </vertical>
+          </scan>
+          <range>
+            <min>${min_range}</min>
+            <max>${max_range}</max>
+            <resolution>0.001</resolution>
+          </range>
+          <noise>
+            <type>gaussian</type>
+            <mean>0.0</mean>
+            <stddev>0.0</stddev>
+          </noise>
+        </ray>
+        <plugin name="gazebo_ros_laser_controller" filename="libgazebo_ros_velodyne_laser.so">
+          <topicName>${ros_topic}</topicName>
+          <frameName>${name}_frame</frameName>
+          <min_range>${min_range}</min_range>
+          <max_range>${max_range}</max_range>
+          <gaussianNoise>0.008</gaussianNoise>
+        </plugin>
+      </sensor>
       </gazebo>
     </xacro:macro>
-    <xacro:macro name="hokuyo_utm30lx_gpu" params="name parent *origin ros_topic update_rate ray_count min_angle max_angle">
-      <xacro:hokuyo_utm30lx_model name="${name}" parent="${parent}">
+    <xacro:macro name="vlp16_gpu" params="name parent *origin ros_topic update_rate ray_count min_angle max_angle">
+      <xacro:vlp16_model name="${name}" parent="${parent}">
         <xacro:insert_block name="origin" />
-      </xacro:hokuyo_utm30lx_model>
+      </xacro:vlp16_model>
       <gazebo reference="${name}_frame">
         <sensor type="gpu_ray" name="${name}">

File: hector_xacro_tools/urdf/joint_macros.urdf.xacro (robot description, xacro)
@@ -1,12 +1,12 @@
 <?xml version="1.0"?>
-<robot xmlns:xacro="http://www.ros.org/wiki/xacro">
+<robot xmlns:xacro="http://ros.org/wiki/xacro">
   <xacro:macro name="joint_standard_transmission" params="name">
     <transmission name="${name}_joint_transmission">
       <type>transmission_interface/SimpleTransmission</type>
       <joint name="${name}">
-        <hardwareInterface>EffortJointInterface</hardwareInterface>
+        <hardwareInterface>hardware_interface/EffortJointInterface</hardwareInterface>
       </joint>
       <actuator name="${name}_joint_motor">
-        <hardwareInterface>EffortJointInterface</hardwareInterface>
+        <hardwareInterface>hardware_interface/EffortJointInterface</hardwareInterface>
         <mechanicalReduction>1</mechanicalReduction>
       </actuator>
