Commit message: Imported upstream version '0.5.1' of 'upstream'

File: hector_sensors_description/urdf/camera360.urdf.xacro (robot description, xacro)
@@ -1,7 +1,9 @@
 <?xml version="1.0"?>
-<robot xmlns:xacro="http://ros.org/wiki/xacro">
+<robot xmlns:xacro="http://www.ros.org/wiki/xacro">
   <xacro:property name="M_PI" value="3.1415926535897931" />
-  <xacro:property name="dist_between_cameras" value="0.03850784" />
-  <xacro:macro name="camera360" params="name right_cam_name left_cam_name parent *origin *calibration ros_topic update_rate res_x res_y image_format fov">
+  <xacro:property name="default_collision_radius" value="0.025" />
+  <xacro:property name="visual_radius" value="0.02" />
+  <xacro:property name="cable_collision_length" value="0.05" />
+  <xacro:macro name="camera360" params="name right_cam_name left_cam_name parent collision_radius:=${default_collision_radius} *origin *calibration dist_between_cameras ros_topic update_rate res_x res_y image_format fov">
     <joint name="${name}_center_joint" type="fixed">
       <xacro:insert_block name="origin" />
@@ -9,7 +11,46 @@
       <child link="${name}_center_link"/>
     </joint>
-    <link name="${name}_center_link" />
+    <link name="${name}_center_link">
+      <!-- Sphere body -->
+      <visual>
+        <origin xyz="0 0 0" rpy="0 0 0"/>
+        <geometry>
+          <sphere radius="${visual_radius}"/>
+        </geometry>
+        <material name="Grey">
+          <color rgba="0.5 0.5 0.5 1"/>
+        </material>
+      </visual>
+      <collision>
+        <origin xyz="0 0 0" rpy="0 0 0"/>
+        <geometry>
+          <sphere radius="${collision_radius}"/>
+        </geometry>
+        <material name="Grey">
+          <color rgba="0.5 0.5 0.5 1"/>
+        </material>
+      </collision>
+      <!-- Cable -->
+<!--      <visual>
+        <origin xyz="${visual_radius + cable_collision_length/2} 0 0" rpy="0 0 0"/>
+        <geometry>
+          <box size="${cable_collision_length} 0.03 0.03"/>
+        </geometry>
+        <material name="Grey">
+          <color rgba="0.5 0.5 0.5 1"/>
+        </material>
+      </visual>-->
+      <collision>
+        <origin xyz="${0.011 + cable_collision_length/2} 0 0" rpy="0 0 0"/>
+        <geometry>
+          <box size="${cable_collision_length} 0.03 0.03"/>
+        </geometry>
+        <material name="Grey">
+          <color rgba="0.5 0.5 0.5 1"/>
+        </material>
+      </collision>
+    </link>
     <joint name="${name}_${right_cam_name}_joint" type="fixed">
-      <origin xyz="${0} ${dist_between_cameras/2} 0" rpy="${M_PI*0.5} 0 ${-M_PI*0.5}"/>
+      <origin xyz="0 ${dist_between_cameras/2} 0" rpy="${M_PI*0.5} 0 ${-M_PI*0.5}"/>
       <parent link="${name}_center_link"/>
       <child link="${name}_${right_cam_name}_link"/>
@@ -38,4 +79,16 @@
           </clip>
           <lens>
+            <!--
+            Crashes gazebo on some machines, so revert for now
+            <type>custom</type>
+            <custom_function>
+              <c1>2</c1>
+              <c2>2</c2>
+              <f>1.0</f>
+              <fun>sin</fun>
+            </custom_function>
+            <cutoff_angle>${fov/2}</cutoff_angle>
+            <env_texture_size>1024</env_texture_size>
+            -->
             <type>stereographic</type>
             <scale_to_hfov>true</scale_to_hfov>
@@ -59,5 +112,5 @@
     <link name="${name}_${left_cam_name}_optical_frame"/>
     <joint name="${name}_${left_cam_name}_joint" type="fixed">
-      <origin xyz="0 0 0" rpy="${M_PI/2} 0.0 ${M_PI/2}" />
+      <origin xyz="0 0 0" rpy="0 ${-M_PI/2} ${M_PI/2}" />
       <parent link="${name}_${left_cam_name}_optical_frame"/>
       <child link="${name}_${left_cam_name}_link" />
@@ -80,4 +133,16 @@
           </clip>
           <lens>
+            <!--
+            Crashes gazebo on some machines, so revert for now
+            <type>custom</type>
+            <custom_function>
+              <c1>2</c1>
+              <c2>2</c2>
+              <f>1.0</f>
+              <fun>sin</fun>
+            </custom_function>
+            <cutoff_angle>${fov/2}</cutoff_angle>
+            <env_texture_size>1024</env_texture_size>
+            -->
             <type>stereographic</type>
             <scale_to_hfov>true</scale_to_hfov>

File: hector_sensors_description/urdf/flir_a35_camera.urdf.xacro (robot description, xacro)
@@ -1,5 +1,6 @@
 <?xml version="1.0"?>
-<robot xmlns:xacro="http://ros.org/wiki/xacro">
+<robot xmlns:xacro="http://www.ros.org/wiki/xacro">
   <xacro:include filename="$(find hector_xacro_tools)/urdf/sensor_macros.urdf.xacro" />
+  <!--Dimensions taken from http://www.flir.com/automation/display/?id=56341-->
   <xacro:macro name="flir_a35_camera_model" params="name parent *origin">
     <joint name="${name}_joint" type="fixed">
@@ -11,8 +12,8 @@
       <xacro:inertial_sphere mass="0.01" diameter="0.07" />
       <visual>
-        <origin xyz="${0.106*-0.5} 0 0" rpy="0 0 0" />
+        <origin xyz="${0.072*-0.5 - 0.0184} 0 0" rpy="0 0 0" />
         <geometry>
-          <!--Dimensions taken from http://www.flir.com/automation/display/?id=56341-->
-          <box size="0.106 0.04 0.043" />
+          <!-- Rear cap: 13.7mm, front cap: 18.4, body length: 72mm, body width: 40mm, body height: 43mm -->
+          <mesh filename="package://hector_sensors_description/meshes/flir_a35_camera/flir_a35_housing.stl" scale="1.0 1.0 1.0"/>
         </geometry>
         <material name="DarkGrey">
@@ -21,8 +22,7 @@
       </visual>
       <collision>
-        <origin xyz="${0.106*-0.5} 0 0" rpy="0 0 0" />
+        <origin xyz="${0.1041*-0.5} 0 0" rpy="0 0 0" />
         <geometry>
-          <!--Dimensions taken from http://www.flir.com/automation/display/?id=56341-->
-          <box size="0.106 0.04 0.043" />
+          <box size="0.1041 0.04 0.043" />
         </geometry>
       </collision>

File: hector_sensors_description/urdf/generic_thermal_camera.urdf.xacro (robot description, xacro)
@@ -1,6 +1,6 @@
 <?xml version="1.0"?>
-<robot xmlns:xacro="http://ros.org/wiki/xacro">
+<robot xmlns:xacro="http://www.ros.org/wiki/xacro">
   <xacro:include filename="$(find hector_xacro_tools)/urdf/sensor_macros.urdf.xacro" />
-  <xacro:macro name="generic_thermal_camera" params="name parent *origin">
+  <xacro:macro name="generic_thermal_camera" params="name parent resolution_x:=320 resolution_y:=256 *origin">
     <joint name="${name}_joint" type="fixed">
       <xacro:insert_block name="origin" />
@@ -9,17 +9,4 @@
     </joint>
     <link name="${name}_frame">
-      <!--        <xacro:inertial_sphere mass="0.01" diameter="0.07" />
-      <visual>
-      <origin xyz="0 0 0" rpy="0 0 0" />
-      <geometry>
-      <mesh filename="package://hector_sensors_description/meshes/thermaleye_camera/thermaleye_camera_hector_v2.dae"/>
-      </geometry>
-      </visual>
-      <collision>
-      <origin xyz="0 0 0" rpy="0 0 0" />
-      <geometry>
-      <mesh filename="package://hector_sensors_description/meshes/thermaleye_camera/thermaleye_camera_hector_v2.stl"/>
-      </geometry>
-      </collision>-->
     </link>
     <xacro:add_optical_frame name="${name}" />
@@ -31,6 +18,6 @@
           <image>
             <format>R8G8B8</format>
-            <width>320</width>
-            <height>256</height>
+            <width>${resolution_x}</width>
+            <height>${resolution_y}</height>
           </image>
           <clip>

File: hector_sensors_description/urdf/realsense_d435_camera.urdf.xacro (robot description, xacro)
@@ -8,11 +8,20 @@
   <node pkg="tf" type="static_transform_publisher" name="kinect_base_link2" args="0 0 0 -1.57 0 -1.57 /arm_rgbd_cam_depth_frame /arm_rgbd_cam_depth_optical_frame  100" />
 -->
-<robot xmlns:xacro="http://ros.org/wiki/xacro">
-    <xacro:property name="M_PI" value="3.1415926535897931" />
+<robot xmlns:xacro="http://www.ros.org/wiki/xacro">
+  <xacro:property name="M_PI" value="3.1415926535897931" />
+  <xacro:property name="realsense_d435_width" value="0.09"/>
+  <xacro:property name="realsense_d435_height" value="0.025"/>
+  <xacro:property name="realsense_d435_depth" value="0.025"/>
+  <xacro:property name="realsense_d435_front_to_depth" value="0.0042" /> <!-- Intel_RealSense_D400_Family_Datasheet_Jan2019.pdf, page 64 -->
+  <xacro:property name="realsense_d435_mount_hole_to_front" value="0.0149" /> <!-- Measured from CAD file -->
+  <xacro:property name="realsense_d435_case_offset_x" value="${realsense_d435_front_to_depth - realsense_d435_depth/2.0}"/>
+  <xacro:property name="realsense_d435_case_offset_y" value="-0.0175"/> <!-- mounting hole to depth frame, Intel_RealSense_D400_Family_Datasheet_Jan2019.pdf, page 66 -->
+  <xacro:property name="realsense_d435_case_offset_z" value="0.0"/>
     <!--
-     This macro only adds the model, it does not also add
-     the openni gazebo plugin. See the 'asus_camera' macro below for that
+     This macro only adds the model, it does not also add the openni gazebo plugin.
+     The origin is the left infrared (depth) camera, which is also the origin of the depth image
     -->
     <xacro:macro name="realsense_d435_camera_model" params="name parent *origin">
+      <xacro:arg name="add_raycast_self_filter_geom" default="false"/>
       <joint name="${name}_joint" type="fixed">
         <xacro:insert_block name="origin" />
@@ -26,25 +35,41 @@
           <inertia ixx="5.8083e-4" ixy="0" ixz="0" iyy="3.0833e-5" iyz="0" izz="5.9083e-4" />
         </inertial>
-        <visual>
-          <origin xyz="0 0.0115 0" rpy="0 0 0" />
+	<visual>
+          <origin xyz="${realsense_d435_front_to_depth} ${realsense_d435_case_offset_y} 0.0" rpy="${M_PI/2} 0 ${M_PI/2}" />
+          <geometry>
+            <mesh filename="package://hector_sensors_description/meshes/intel_realsense_d435/D435.dae" scale="0.001 0.001 0.001" />
+          </geometry>
+        </visual>
+        <collision>
+          <origin xyz="${realsense_d435_case_offset_x} ${realsense_d435_case_offset_y} ${realsense_d435_case_offset_z}" rpy="0 0 0" />
           <geometry>
             <!--Dimensions taken from https://click.intel.com/intelr-realsensetm-depth-camera-d435.html-->
-            <box size="0.025 0.09 0.025" />
+            <box size="${realsense_d435_depth} ${realsense_d435_width} ${realsense_d435_height}" />
           </geometry>
-          <material name="DarkGrey">
-            <color rgba="0.3 0.3 0.3 1"/>
-          </material>
-        </visual>
+        </collision>
+      <xacro:if value="$(arg add_raycast_self_filter_geom)">
         <collision>
-          <origin xyz="0 0.0115 0" rpy="0 0 0" />
+          <origin xyz="${realsense_d435_case_offset_x} ${realsense_d435_case_offset_y} ${realsense_d435_case_offset_z}" rpy="${M_PI*0.5} 0 0" />
           <geometry>
-            <!--Dimensions taken from https://click.intel.com/intelr-realsensetm-depth-camera-d435.html-->
-            <box size="0.025 0.09 0.025" />
-          </geometry>update_rate
+            <cylinder length="0.09" radius="0.0177"/>
+          </geometry>
         </collision>
+      </xacro:if>
       </link>
       <gazebo reference="${name}_link">
         <material>Gazebo/Grey</material>
       </gazebo>
+    </xacro:macro>
+    <xacro:macro name="realsense_d435_camera_model_with_mount" params="name parent *origin">
+      <joint name="${name}_mount_joint" type="fixed">
+        <xacro:insert_block name="origin" />
+        <parent link="${parent}"/>
+        <child link="${name}_mount_link"/>
+      </joint>
+      <link name="${name}_mount_link">
+      </link>
+      <xacro:realsense_d435_camera_model name="${name}" parent="${name}_mount_link">
+        <origin xyz="${realsense_d435_mount_hole_to_front - realsense_d435_front_to_depth} ${-realsense_d435_case_offset_y} ${realsense_d435_height/2.0}" rpy="0 0 0"/>
+      </xacro:realsense_d435_camera_model>
     </xacro:macro>
     <xacro:macro name="realsense_d435_camera_model_no_geom" params="name parent *origin">
@@ -65,5 +90,5 @@
             <image>
               <format>B8G8R8</format>
-              <width>848</width>
+              <width>640</width>
               <height>480</height>
             </image>
@@ -75,10 +100,10 @@
           <plugin name="${name}_camera_controller" filename="libgazebo_ros_openni_kinect.so">
             <cameraName>${name}</cameraName>
-            <imageTopicName>rgb/${image_topic}</imageTopicName>
-            <cameraInfoTopicName>rgb/camera_info</cameraInfoTopicName>
+            <imageTopicName>color/${image_topic}</imageTopicName>
+            <cameraInfoTopicName>color/camera_info</cameraInfoTopicName>
             <depthImageTopicName>depth/image_raw</depthImageTopicName>
             <depthImageCameraInfoTopicName>depth/camera_info</depthImageCameraInfoTopicName>
             <pointCloudTopicName>${depth_points_topic}</pointCloudTopicName>
-            <frameName>${name}_depth_optical_frame</frameName>
+            <frameName>${name}_color_optical_frame</frameName>
           </plugin>
         </sensor>
@@ -87,4 +112,5 @@
     <!--
       Use the macro below for adding the realsense model with link geometry
+      The origin is the left infrared (depth) camera, which is also the origin of the depth image
     -->
     <xacro:macro name="realsense_d435_camera" params="name parent *origin">
@@ -92,5 +118,14 @@
         <xacro:insert_block name="origin" />
       </xacro:realsense_d435_camera_model>
-      <xacro:realsense_d435_camera_gazebo_plugin_macro name="${name}" parent="${parent}" image_topic="rgb/image_raw" depth_points_topic="depth/points" min_range="0.3" max_range="9.0" update_rate="20"/>
+      <xacro:realsense_d435_camera_gazebo_plugin_macro name="${name}" parent="${parent}" image_topic="image_raw" depth_points_topic="depth/points" min_range="0.3" max_range="9.0" update_rate="20"/>
+    </xacro:macro>
+    <!--
+      Insert the realsense with link geometry. Origin is the mounting hole at the back of the camera.
+    -->
+    <xacro:macro name="realsense_d435_camera_with_mount" params="name parent *origin">
+      <xacro:realsense_d435_camera_model_with_mount name="${name}" parent="${parent}">
+        <xacro:insert_block name="origin" />
+      </xacro:realsense_d435_camera_model_with_mount>
+      <xacro:realsense_d435_camera_gazebo_plugin_macro name="${name}" parent="${parent}" image_topic="image_raw" depth_points_topic="depth/points" min_range="0.3" max_range="9.0" update_rate="20"/>
     </xacro:macro>
     <!--
@@ -102,5 +137,5 @@
         <xacro:insert_block name="origin" />
       </xacro:realsense_d435_camera_model_no_geom>
-      <xacro:realsense_camera_gazebo_plugin_macro name="${name}" parent="${parent}" image_topic="rgb/image_raw" depth_points_topic="depth/points" min_range="0.3" max_range="9.0" update_rate="20"/>
+      <xacro:realsense_camera_gazebo_plugin_macro name="${name}" parent="${parent}" image_topic="image_raw" depth_points_topic="depth/points" min_range="0.3" max_range="9.0" update_rate="20"/>
     </xacro:macro>
     <xacro:macro name="realsense_d435_camera_no_geom_comprehensive_params" params="name parent *origin image_topic depth_points_topic min_range max_range update_rate">
@@ -116,3 +151,9 @@
       <xacro:realsense_d435_camera_gazebo_plugin_macro name="${name}" parent="${parent}" image_topic="${image_topic}" depth_points_topic="${depth_points_topic}" min_range="${min_range}" max_range="${max_range}" update_rate="${update_rate}"/>
     </xacro:macro>
+    <xacro:macro name="realsense_d435_camera_with_mount_comprehensive_params" params="name parent *origin image_topic depth_points_topic min_range max_range update_rate">
+      <xacro:realsense_d435_camera_model_with_mount name="${name}" parent="${parent}">
+        <xacro:insert_block name="origin" />
+      </xacro:realsense_d435_camera_model_with_mount>
+      <xacro:realsense_d435_camera_gazebo_plugin_macro name="${name}" parent="${parent}" image_topic="${image_topic}" depth_points_topic="${depth_points_topic}" min_range="${min_range}" max_range="${max_range}" update_rate="${update_rate}"/>
+    </xacro:macro>
   </robot>

File: hector_sensors_description/urdf/ricoh_theta.urdf.xacro (robot description, xacro)
@@ -1,11 +1,11 @@
 <?xml version="1.0"?>
-<robot xmlns:xacro="http://ros.org/wiki/xacro">
+<robot xmlns:xacro="http://www.ros.org/wiki/xacro">
   <xacro:property name="M_PI" value="3.1415926535897931" />
   <xacro:property name="theta_dist_between_cameras" value="0.01602869966119076" />
   <xacro:macro name="ricoh_theta_camera" params="name cam_front_name cam_rear_name parent *origin ros_topic cam_info_topic update_rate res_x res_y image_format fov">
-    <joint name="ricoh_theta_center_joint" type="fixed">
+    <joint name="${name}_center_joint" type="fixed">
       <xacro:insert_block name="origin" />
       <parent link="${parent}"/>
-      <child link="ricoh_theta_center_link"/>
+      <child link="${name}_center_link"/>
     </joint>
     <link name="${name}_center_link" />
