Commit message: Imported upstream version '0.5.1' of 'upstream'

File: hector_sensors_description/urdf/vlp16.urdf.xacro (robot description, xacro)
@@ -1,68 +1,59 @@
 <?xml version="1.0"?>
-<robot xmlns:xacro="http://ros.org/wiki/xacro">
-    <xacro:property name="M_PI" value="3.1415926535897931" />
-    <xacro:macro name="vlp16_model" params="name parent *origin">
-      <joint name="${name}_joint" type="fixed">
-        <xacro:insert_block name="origin" />
-        <parent link="${parent}"/>
-        <child link="${name}_frame"/>
-      </joint>
-      <link name="${name}_frame">
-        <xacro:inertial_sphere mass="0.8" diameter="0.1033" />
-        <visual>        -->
-          <origin rpy="0 0 0" xyz="0 0 0.0018500"/>
-          <geometry>
-            <cylinder radius="0.0516" length="0.0717"/>
-          </geometry>
-        </visual>
-        <collision>
-          <origin rpy="0 0 0" xyz="0 0 0.0018500"/>
-          <geometry>
-            <cylinder radius="0.0516" length="0.0717"/>
-          </geometry>
-        </collision>
-      </link>
-    </xacro:macro>
-    <xacro:macro name="vlp16" params="name parent *origin ros_topic">
-      <xacro:vlp16_advanced_parameters name="${name}" parent="${parent}" ros_topic="${ros_topic}" update_rate="10" horizontal_samples="512" vertical_samples="8" min_range="0.45" max_range="100">
-        <xacro:insert_block name="origin" />
-      </xacro:vlp16_advanced_parameters>
-    </xacro:macro>
-    <xacro:macro name="vlp16_advanced_parameters" params="name parent *origin ros_topic update_rate horizontal_samples vertical_samples min_range max_range">
-      <xacro:vlp16_model name="${name}" parent="${parent}">
-        <xacro:insert_block name="origin" />
-      </xacro:vlp16_model>
-      <gazebo reference="${name}_frame">
-<!--        <sensor type="ray" name="${name}">
-          <always_on>true</always_on>
-          <update_rate>${update_rate}</update_rate>
-          <pose>0 0 0 0 0 0</pose>
-          <visualize>false</visualize>
-          <ray>
-            <scan>
-              <horizontal>
-                <samples>${ray_count}</samples>
-                <resolution>1</resolution>
-                <min_angle>${min_angle * M_PI/180}</min_angle>
-                <max_angle>${max_angle * M_PI/180}</max_angle>
-              </horizontal>
-            </scan>
-            <range>
-              <min>0.2</min>
-              <max>30.0</max>
-              <resolution>0.01</resolution>
-            </range>
-            <noise>
-              <type>gaussian</type>
-              <mean>0.0</mean>
-              <stddev>0.004</stddev>
-            </noise>
-          </ray>
-          <plugin name="gazebo_ros_${name}_controller" filename="libgazebo_ros_laser.so">
-            <topicName>${ros_topic}</topicName>
-            <frameName>${name}_frame</frameName>
-          </plugin>
-        </sensor>-->
-      <sensor type="ray" name="${name}-VLP16">
+<robot xmlns:xacro="http://www.ros.org/wiki/xacro">
+  <xacro:include filename="$(find hector_xacro_tools)/urdf/inertia_tensors.urdf.xacro"/>
+  <xacro:property name="M_PI" value="3.1415926535897931"/>
+  <xacro:macro name="vlp16_model" params="name parent *origin">
+    <joint name="${name}_joint" type="fixed">
+      <xacro:insert_block name="origin"/>
+      <parent link="${parent}"/>
+      <child link="${name}_frame"/>
+    </joint>
+    <link name="${name}_frame">
+      <xacro:inertial_sphere mass="0.83" diameter="0.1033"/>
+      <visual>
+        <origin xyz="0 0 -0.0378" rpy="${M_PI/2} 0 ${M_PI}"/>
+        <geometry>
+          <mesh filename="package://hector_sensors_description/meshes/vlp16/VLP16_base_1.dae" scale="0.001 0.001 0.001"/>
+        </geometry>
+      </visual>
+      <visual>
+        <origin xyz="0 0 -0.0378" rpy="${M_PI/2} 0 ${M_PI}"/>
+        <geometry>
+          <mesh filename="package://hector_sensors_description/meshes/vlp16/VLP16_base_2.dae" scale="0.001 0.001 0.001"/>
+        </geometry>
+      </visual>
+      <visual>
+        <origin xyz="0 0 -0.0378" rpy="${M_PI/2} 0 ${M_PI}"/>
+        <geometry>
+          <mesh filename="package://hector_sensors_description/meshes/vlp16/VLP16_scan.dae" scale="0.001 0.001 0.001"/>
+        </geometry>
+      </visual>
+      <collision>
+        <origin rpy="0 0 0" xyz="0 0 -0.00225"/>
+        <geometry>
+          <cylinder radius="0.0516" length="0.0717"/>
+        </geometry>
+      </collision>
+    </link>
+  </xacro:macro>
+  <xacro:macro name="vlp16" params="name parent *origin ros_topic">
+    <xacro:vlp16_advanced_parameters name="${name}" parent="${parent}" ros_topic="${ros_topic}" update_rate="10" horizontal_samples="512" vertical_samples="8" min_range="0.45" max_range="100">
+      <xacro:insert_block name="origin"/>
+    </xacro:vlp16_advanced_parameters>
+  </xacro:macro>
+  <xacro:macro name="vlp16_advanced_parameters" params="name parent *origin ros_topic update_rate horizontal_samples vertical_samples min_range max_range use_gpu:='false'">
+    <xacro:vlp16_model name="${name}" parent="${parent}">
+      <xacro:insert_block name="origin"/>
+    </xacro:vlp16_model>
+    <gazebo reference="${name}_frame">
+      <xacro:if value="${use_gpu}">
+        <xacro:property name="sensor_type" value="gpu_ray"/>
+        <xacro:property name="gazebo_plugin_name" value="libgazebo_ros_velodyne_gpu_laser.so"/>
+      </xacro:if >
+      <xacro:unless value="${use_gpu}">
+        <xacro:property name="sensor_type" value="ray"/>
+        <xacro:property name="gazebo_plugin_name" value="libgazebo_ros_velodyne_laser.so"/>
+      </xacro:unless>
+      <sensor type="${sensor_type}" name="${name}-VLP16">
         <pose>0 0 0 0 0 0</pose>
         <visualize>false</visualize>
@@ -74,5 +65,5 @@
               <resolution>1</resolution>
               <min_angle>-${M_PI}</min_angle>
-              <max_angle> ${M_PI}</max_angle>
+              <max_angle>${M_PI}</max_angle>
             </horizontal>
             <vertical>
@@ -80,5 +71,5 @@
               <resolution>1</resolution>
               <min_angle>-${15.0*M_PI/180.0}</min_angle>
-              <max_angle> ${15.0*M_PI/180.0}</max_angle>
+              <max_angle>${15.0*M_PI/180.0}</max_angle>
             </vertical>
           </scan>
@@ -94,5 +85,5 @@
           </noise>
         </ray>
-        <plugin name="gazebo_ros_laser_controller" filename="libgazebo_ros_velodyne_laser.so">
+        <plugin name="gazebo_ros_laser_controller" filename="${gazebo_plugin_name}">
           <topicName>${ros_topic}</topicName>
           <frameName>${name}_frame</frameName>
@@ -102,41 +93,5 @@
         </plugin>
       </sensor>
-      </gazebo>
-    </xacro:macro>
-    <xacro:macro name="vlp16_gpu" params="name parent *origin ros_topic update_rate ray_count min_angle max_angle">
-      <xacro:vlp16_model name="${name}" parent="${parent}">
-        <xacro:insert_block name="origin" />
-      </xacro:vlp16_model>
-      <gazebo reference="${name}_frame">
-        <sensor type="gpu_ray" name="${name}">
-          <update_rate>${update_rate}</update_rate>
-          <pose>0 0 0 0 0 0</pose>
-          <visualize>false</visualize>
-          <ray>
-            <scan>
-              <horizontal>
-                <samples>${ray_count}</samples>
-                <resolution>1</resolution>
-                <min_angle>${min_angle * M_PI/180}</min_angle>
-                <max_angle>${max_angle * M_PI/180}</max_angle>
-              </horizontal>
-            </scan>
-            <range>
-              <min>0.2</min>
-              <max>30.0</max>
-              <resolution>0.01</resolution>
-            </range>
-            <noise>
-              <type>gaussian</type>
-              <mean>0.0</mean>
-              <stddev>0.004</stddev>
-            </noise>
-          </ray>
-          <plugin name="gazebo_ros_${name}_controller" filename="libgazebo_ros_gpu_laser.so">
-            <topicName>${ros_topic}</topicName>
-            <frameName>${name}_frame</frameName>
-          </plugin>
-        </sensor>
-      </gazebo>
-    </xacro:macro>
+    </gazebo>
+  </xacro:macro>
 </robot>

File: hector_xacro_tools/urdf/joint_macros.urdf.xacro (robot description, xacro)
@@ -1,4 +1,4 @@
 <?xml version="1.0"?>
-<robot xmlns:xacro="http://ros.org/wiki/xacro">
+<robot xmlns:xacro="http://www.ros.org/wiki/xacro">
   <xacro:macro name="joint_standard_transmission" params="name">
     <transmission name="${name}_joint_transmission">
@@ -16,3 +16,33 @@
     </gazebo>
   </xacro:macro>
+  <xacro:macro name="joint_position_transmission" params="name">
+    <transmission name="${name}_joint_transmission">
+      <type>transmission_interface/SimpleTransmission</type>
+      <joint name="${name}">
+        <hardwareInterface>hardware_interface/PositionJointInterface</hardwareInterface>
+      </joint>
+      <actuator name="${name}_joint_motor">
+        <hardwareInterface>hardware_interface/PositionJointInterface</hardwareInterface>
+        <mechanicalReduction>1</mechanicalReduction>
+      </actuator>
+    </transmission>
+    <gazebo reference="${name}">
+      <implicitSpringDamper>1</implicitSpringDamper>
+    </gazebo>
+  </xacro:macro>
+  <xacro:macro name="joint_velocity_transmission" params="name">
+    <transmission name="${name}_joint_transmission">
+      <type>transmission_interface/SimpleTransmission</type>
+      <joint name="${name}">
+        <hardwareInterface>hardware_interface/VelocityJointInterface</hardwareInterface>
+      </joint>
+      <actuator name="${name}_joint_motor">
+        <hardwareInterface>hardware_interface/VelocityJointInterface</hardwareInterface>
+        <mechanicalReduction>1</mechanicalReduction>
+      </actuator>
+    </transmission>
+    <gazebo reference="${name}">
+      <implicitSpringDamper>1</implicitSpringDamper>
+    </gazebo>
+  </xacro:macro>
 </robot>
