Commit message: Rebase from 'upstream'

File: hector_components_description/urdf/hector_multisensor_head.urdf.xacro (robot description, xacro)
@@ -1,9 +1,9 @@
 <?xml version="1.0"?>
 <robot
-    xmlns:xacro="http://ros.org/wiki/xacro" name="hector_multisensor_head">
+    xmlns:xacro="http://www.ros.org/wiki/xacro" name="hector_multisensor_head">
     <xacro:include filename="$(find hector_xacro_tools)/urdf/inertia_tensors.urdf.xacro"/>
     <xacro:include filename="$(find hector_sensors_description)/urdf/hokuyo_utm30lx.urdf.xacro" />
     <xacro:include filename="$(find hector_sensors_description)/urdf/asus_camera.urdf.xacro" />
-    <property name="M_PI" value="3.14159265359"/>
+    <xacro:property name="M_PI" value="3.14159265359"/>
     <xacro:macro name="hector_multisensor_head_macro" params="parent name scaling *origin">
         <link name="${name}_link">
@@ -12,5 +12,5 @@
             </xacro:inertial_sphere_with_pose>
             <collision name="collision">
-                 <insert_block name="origin"/>
+                 <xacro:insert_block name="origin"/>
                 <geometry>
                     <mesh filename="package://hector_components_description/meshes/hector_multisensor_head/multisensor_head_collision.stl" scale="${scaling} ${scaling} ${scaling}"/>
@@ -18,5 +18,5 @@
             </collision>
             <visual>
-                <insert_block name="origin"/>
+                <xacro:insert_block name="origin"/>
                 <geometry>
                     <mesh filename="package://hector_components_description/meshes/hector_multisensor_head/multisensor_head.stl" scale="${scaling} ${scaling} ${scaling}"/>
@@ -26,5 +26,5 @@
         <joint name="${name}_lidar_spinning_joint" type="continuous">
             <origin xyz="0.061 0.0 0.134" rpy="0 0 0"/>
-            <insert_block name="origin"/>
+            <xacro:insert_block name="origin"/>
             <parent link="${name}_link" />
             <child link="${name}_lidar_mount_link"/>

File: hector_components_description/urdf/spinning_hokuyo_utm30lx.urdf.xacro (robot description, xacro)
@@ -1,22 +1,22 @@
 <?xml version="1.0"?>
-<robot xmlns:xacro="http://playerstage.sourceforge.net/gazebo/xmlschema/#interface">
-  <property name="M_PI" value="3.14159265359"/>
+<robot xmlns:xacro="http://www.ros.org/wiki/xacro">
+  <xacro:property name="M_PI" value="3.14159265359"/>
   <xacro:include filename="$(find hector_components_description)/urdf/spinning_lidar_mount.urdf.xacro"/>
   <xacro:include filename="$(find hector_sensors_description)/urdf/hokuyo_utm30lx.urdf.xacro"/>
-  <macro name="spinning_hokuyo_utm30lx_macro" params="parent name angle_deg *origin">
-    <spinning_lidar_macro parent="${parent}" name="${name}" angle_deg="45">
-      <insert_block name="origin"/>
-    </spinning_lidar_macro>
+  <xacro:macro name="spinning_hokuyo_utm30lx_macro" params="parent name angle_deg *origin">
+    <xacro:spinning_lidar_macro parent="${parent}" name="${name}" angle_deg="45">
+      <xacro:insert_block name="origin"/>
+    </xacro:spinning_lidar_macro>
     <xacro:hokuyo_utm30lx_gpu name="${name}_hokuyo_laser" parent="${name}_spinning_lidar_spin_link" ros_topic="${name}_spinning_lidar/scan" update_rate="40" ray_count="1040" min_angle="-130" max_angle="130">
       <origin xyz="0.00 -0.0 0.055" rpy="0 ${angle_deg * M_PI/180.0} 0"/>
     </xacro:hokuyo_utm30lx_gpu>
-  </macro>
-  <macro name="spinning_hokuyo_utm30lx_lidar_mount_offset_macro" params="parent name scan_topic_in_namespace angle_deg *origin">
-    <spinning_lidar_macro parent="${parent}" name="${name}" angle_deg="45">
-      <insert_block name="origin"/>
-    </spinning_lidar_macro>
+  </xacro:macro>
+  <xacro:macro name="spinning_hokuyo_utm30lx_lidar_mount_offset_macro" params="parent name scan_topic_in_namespace angle_deg *origin">
+    <xacro:spinning_lidar_macro parent="${parent}" name="${name}" angle_deg="45">
+      <xacro:insert_block name="origin"/>
+    </xacro:spinning_lidar_macro>
     <xacro:hokuyo_utm30lx_gpu name="${name}_hokuyo_laser" parent="${name}_spinning_lidar_spin_link" ros_topic="${name}_spinning_lidar/${scan_topic_in_namespace}" update_rate="40" ray_count="1040" min_angle="-130" max_angle="130">
       <origin xyz="0.021 0.0  -0.0  " rpy="0 ${-angle_deg * M_PI/180.0} ${M_PI}"/>
     </xacro:hokuyo_utm30lx_gpu>
-  </macro>
+  </xacro:macro>
 </robot>

Commit message: Imported upstream version '0.4.2' of 'upstream'

File: hector_components_description/urdf/hector_multisensor_head.urdf.xacro (robot description, xacro)
@@ -6,9 +6,10 @@
     <xacro:include filename="$(find hector_sensors_description)/urdf/asus_camera.urdf.xacro" />
     <xacro:property name="M_PI" value="3.14159265359"/>
-    <xacro:macro name="hector_multisensor_head_macro" params="parent name scaling *origin">
+    <xacro:macro name="hector_multisensor_head_macro" params="parent name scaling *origin *calibration">
         <link name="${name}_link">
-            <xacro:inertial_sphere_with_pose mass="0.1" diameter="0.03">
-                <origin xyz="0.0 0.0 0" rpy="0 0 0"/>
-            </xacro:inertial_sphere_with_pose>
+             <inertial>
+	      <mass value="0.8"/>
+	      <inertia ixx="0.0025" ixy="0.0" ixz="0.0001" iyy="0.0013" iyz="0.0" izz="0.0026"/>
+	    </inertial>
             <collision name="collision">
                  <xacro:insert_block name="origin"/>
@@ -26,5 +27,4 @@
         <joint name="${name}_lidar_spinning_joint" type="continuous">
             <origin xyz="0.061 0.0 0.134" rpy="0 0 0"/>
-            <xacro:insert_block name="origin"/>
             <parent link="${name}_link" />
             <child link="${name}_lidar_mount_link"/>
@@ -34,10 +34,10 @@
         </joint>
         <link name="${name}_lidar_mount_link">
-            <xacro:inertial_sphere_with_pose_macro mass="1.1" diameter="0.03">
+            <xacro:inertial_sphere_with_pose_macro mass="0.1" diameter="0.03">
                 <origin xyz="0.0 0.0 0.0" rpy="0 0 0"/>
             </xacro:inertial_sphere_with_pose_macro>
         </link>
         <xacro:hokuyo_utm30lx name="${name}_link_hokuyo_laser" parent="${name}_lidar_mount_link" ros_topic="/head_lidar/scan" update_rate="40" ray_count="1040" min_angle="130" max_angle="-130">
-            <origin xyz="0.0 0.0 0.0" rpy="0 0 0"/>
+            <xacro:insert_block name="calibration" />
         </xacro:hokuyo_utm30lx>
         <transmission name="${name}_lidar_spinning_joint_transmission">
@@ -55,5 +55,5 @@
         </gazebo>
 	<xacro:asus_camera name="${name}_cam" parent="${name}_link">
-	                <origin xyz="0.0385 0.0 0.2385" rpy="0 0 0"/>
+	                <origin xyz="0.065 0.0 0.23" rpy="0 0 0"/>
 	</xacro:asus_camera>
         <!-- <gazebo reference="${name}_spinning_lidar_root_link"><material>Gazebo/Grey</material></gazebo><gazebo reference="${name}_spinning_lidar_spin_link"><material>Gazebo/Grey</material></gazebo> -->
