Commit message: Rebase from 'release/noetic/hector_sensors_description'

File: urdf/parametrized_camera.urdf.xacro (robot description, xacro)
@@ -2,5 +2,5 @@
 <robot xmlns:xacro="http://www.ros.org/wiki/xacro">
   <xacro:property name="M_PI" value="3.1415926535897931" />
-  <xacro:macro name="generic_camera" params="name parent *origin ros_topic cam_info_topic update_rate res_x res_y image_format hfov">
+  <xacro:macro name="parametrized_camera" params="name parent *origin ros_topic cam_info_topic update_rate res_x res_y image_format hfov cx cy k1 k2 k3 t1 t2">
     <joint name="${name}_joint" type="fixed">
       <xacro:insert_block name="origin" />
@@ -50,4 +50,12 @@
             <far>100</far>
           </clip>
+          <distortion>
+            <k1>${k1}</k1>
+            <k2>${k2}</k2>
+            <p1>${t1}</p1>
+            <p2>${t2}</p2>
+            <k3>${k3}</k3>
+            <center>0.5 0.5</center>
+          </distortion>
         </camera>
         <plugin name="${name}_camera_controller" filename="libgazebo_ros_camera.so">
@@ -56,4 +64,11 @@
           <cameraInfoTopicName>${cam_info_topic}</cameraInfoTopicName>
           <frameName>${name}_optical_frame</frameName>
+          <Cx>${cx}</Cx>
+          <Cy>${cy}</Cy>
+          <distortionK1>${k1}</distortionK1>
+          <distortionK2>${k2}</distortionK2>
+          <distortionK3>${k3}</distortionK3>
+          <distortionT1>${t1}</distortionT1>
+          <distortionT2>${t2}</distortionT2>
         </plugin>
       </sensor>
